File: circuit/function_gen_output.kicad_sch (KiCad schematic)
At the start: 6 parts, among them J1 Vin, U1 NE5532

Commit message: Add software files
Signed-off-by: Atharva Lele <itsatharva@gmail.com>
Parts:
- added C1: 10pF, symbol Device:C
- added J2: Output, symbol Connector:Conn_01x01_Male
- added R5: 100k, symbol Device:R_US
Connections:
- net GND: now also C1.2
- net at R4.2, U1.1: now also R5.1
- new net: C1.1, J2.1 (Pin_1), R5.2
Other:
- moved on the sheet: U1C
Changed lines of the file:
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@@
 (kicad_sch (version 20211123) (generator eeschema)
   (paper "A4")
+  (junction (at 147.32 76.2) (diameter 0) (color 0 0 0 0)
+  )
   (junction (at 118.11 68.58) (diameter 0) (color 0 0 0 0)
   )
   (junction (at 118.11 86.36) (diameter 0) (color 0 0 0 0)
   )
+  (junction (at 163.83 76.2) (diameter 0) (color 0 0 0 0)
+  )
   (wire (pts (xy 118.11 86.36) (xy 118.11 78.74))
     (stroke (width 0) (type default) (color 0 0 0 0))
@@
     (stroke (width 0) (type default) (color 0 0 0 0))
   )
+  (wire (pts (xy 163.83 83.82) (xy 163.83 88.9))
+    (stroke (width 0) (type default) (color 0 0 0 0))
+  )
   (wire (pts (xy 118.11 91.44) (xy 118.11 86.36))
     (stroke (width 0) (type default) (color 0 0 0 0))
@@
     (stroke (width 0) (type default) (color 0 0 0 0))
   )
+  (wire (pts (xy 147.32 76.2) (xy 151.13 76.2))
+    (stroke (width 0) (type default) (color 0 0 0 0))
+  )
   (wire (pts (xy 111.76 86.36) (xy 118.11 86.36))
     (stroke (width 0) (type default) (color 0 0 0 0))
@@
     (stroke (width 0) (type default) (color 0 0 0 0))
   )
-  (wire (pts (xy 80.01 24.13) (xy 71.12 24.13))
+  (wire (pts (xy 101.6 33.02) (xy 92.71 33.02))
     (stroke (width 0) (type default) (color 0 0 0 0))
   )
@@
     (stroke (width 0) (type default) (color 0 0 0 0))
   )
-  (wire (pts (xy 80.01 43.18) (xy 71.12 43.18))
-    (stroke (width 0) (type default) (color 0 0 0 0))
-  )
-  (wire (pts (xy 80.01 39.37) (xy 80.01 43.18))
+  (wire (pts (xy 158.75 76.2) (xy 163.83 76.2))
+    (stroke (width 0) (type default) (color 0 0 0 0))
+  )
+  (wire (pts (xy 101.6 52.07) (xy 92.71 52.07))
+    (stroke (width 0) (type default) (color 0 0 0 0))
+  )
+  (wire (pts (xy 101.6 48.26) (xy 101.6 52.07))
     (stroke (width 0) (type default) (color 0 0 0 0))
   )
@@
   )
   (wire (pts (xy 118.11 55.88) (xy 118.11 68.58))
+    (stroke (width 0) (type default) (color 0 0 0 0))
+  )
+  (wire (pts (xy 163.83 76.2) (xy 172.72 76.2))
     (stroke (width 0) (type default) (color 0 0 0 0))
   )
@@
     (pin "2")
   )
-  (symbol (lib_id "Amplifier_Operational:NE5532") (at 82.55 31.75 0) (unit 3)
-    (in_bom yes) (on_board yes) (fields_autoplaced)
-    (property "Reference" "U1" (id 0) (at 81.28 30.4799 0)
+  (symbol (lib_id "Amplifier_Operational:NE5532") (at 104.14 40.64 0) (unit 3)
+    (in_bom yes) (on_board yes) (fields_autoplaced)
+    (property "Reference" "U1" (id 0) (at 102.87 39.3699 0)
       (effects (font (size 1.27 1.27)) (justify left))
     )
-    (property "Value" "NE5532" (id 1) (at 81.28 33.0199 0)
+    (property "Value" "NE5532" (id 1) (at 102.87 41.9099 0)
       (effects (font (size 1.27 1.27)) (justify left))
     )
-    (property "Footprint" "" (id 2) (at 82.55 31.75 0)
-      (effects (font (size 1.27 1.27)) hide)
-    )
-    (property "Datasheet" "http://www.ti.com/lit/ds/symlink/ne5532.pdf" (id 3) (at 82.55 31.75 0)
+    (property "Footprint" "" (id 2) (at 104.14 40.64 0)
+      (effects (font (size 1.27 1.27)) hide)
+    )
+    (property "Datasheet" "http://www.ti.com/lit/ds/symlink/ne5532.pdf" (id 3) (at 104.14 40.64 0)
       (effects (font (size 1.27 1.27)) hide)
     )
@@
     (pin "8")
   )
+  (symbol (lib_id "Connector:Conn_01x01_Male") (at 177.8 76.2 180) (unit 1)
+    (in_bom yes) (on_board yes) (fields_autoplaced)
+    (property "Reference" "J2" (id 0) (at 177.165 71.12 0))
+    (property "Value" "Output" (id 1) (at 177.165 73.66 0))
+    (property "Footprint" "" (id 2) (at 177.8 76.2 0)
+      (effects (font (size 1.27 1.27)) hide)
+    )
+    (property "Datasheet" "~" (id 3) (at 177.8 76.2 0)
+      (effects (font (size 1.27 1.27)) hide)
+    )
+    (pin "1")
+  )
+  (symbol (lib_id "Device:C") (at 163.83 80.01 0) (unit 1)
+    (in_bom yes) (on_board yes) (fields_autoplaced)
+    (property "Reference" "C1" (id 0) (at 167.64 78.7399 0)
+      (effects (font (size 1.27 1.27)) (justify left))
+    )
+    (property "Value" "10pF" (id 1) (at 167.64 81.2799 0)
+      (effects (font (size 1.27 1.27)) (justify left))
+    )
+    (property "Footprint" "" (id 2) (at 164.7952 83.82 0)
+      (effects (font (size 1.27 1.27)) hide)
+    )
+    (property "Datasheet" "~" (id 3) (at 163.83 80.01 0)
+      (effects (font (size 1.27 1.27)) hide)
+    )
+    (pin "1")
+    (pin "2")
+  )
   (symbol (lib_id "power:+5V") (at 90.17 82.55 0) (unit 1)
     (in_bom yes) (on_board yes) (fields_autoplaced)
@@
     )
     (pin "1")
+  )
+  (symbol (lib_id "Device:R_US") (at 154.94 76.2 90) (unit 1)
+    (in_bom yes) (on_board yes) (fields_autoplaced)
+    (property "Reference" "R5" (id 0) (at 154.94 69.85 90))
+    (property "Value" "100k" (id 1) (at 154.94 72.39 90))
+    (property "Footprint" "" (id 2) (at 155.194 75.184 90)
+      (effects (font (size 1.27 1.27)) hide)
+    )
+    (property "Datasheet" "~" (id 3) (at 154.94 76.2 0)
+      (effects (font (size 1.27 1.27)) hide)
+    )
+    (pin "1")
+    (pin "2")
   )
   (symbol (lib_id "Amplifier_Operational:NE5532") (at 130.81 76.2 0) (unit 1)
@@
     (pin "2")
   )
+  (symbol (lib_id "power:GND") (at 163.83 88.9 0) (unit 1)
+    (in_bom yes) (on_board yes) (fields_autoplaced)
+    (property "Reference" "#PWR?" (id 0) (at 163.83 95.25 0)
+      (effects (font (size 1.27 1.27)) hide)
+    )
+    (property "Value" "GND" (id 1) (at 163.83 93.98 0))
+    (property "Footprint" "" (id 2) (at 163.83 88.9 0)
+      (effects (font (size 1.27 1.27)) hide)
+    )
+    (property "Datasheet" "" (id 3) (at 163.83 88.9 0)
+      (effects (font (size 1.27 1.27)) hide)
+    )
+    (pin "1")
+  )
   (symbol (lib_id "Connector:Conn_01x01_Male") (at 85.09 68.58 0) (unit 1)
     (in_bom yes) (on_board yes)
@@
     (pin "1")
   )
-  (symbol (lib_id "power:+5V") (at 71.12 24.13 0) (unit 1)
-    (in_bom yes) (on_board yes) (fields_autoplaced)
-    (property "Reference" "#PWR?" (id 0) (at 71.12 27.94 0)
-      (effects (font (size 1.27 1.27)) hide)
-    )
-    (property "Value" "+5V" (id 1) (at 71.12 19.05 0))
-    (property "Footprint" "" (id 2) (at 71.12 24.13 0)
-      (effects (font (size 1.27 1.27)) hide)
-    )
-    (property "Datasheet" "" (id 3) (at 71.12 24.13 0)
+  (symbol (lib_id "power:+5V") (at 92.71 33.02 0) (unit 1)
+    (in_bom yes) (on_board yes) (fields_autoplaced)
+    (property "Reference" "#PWR?" (id 0) (at 92.71 36.83 0)
+      (effects (font (size 1.27 1.27)) hide)
+    )
+    (property "Value" "+5V" (id 1) (at 92.71 27.94 0))
+    (property "Footprint" "" (id 2) (at 92.71 33.02 0)
+      (effects (font (size 1.27 1.27)) hide)
+    )
+    (property "Datasheet" "" (id 3) (at 92.71 33.02 0)
       (effects (font (size 1.27 1.27)) hide)
     )
@@
     (pin "2")
   )
-  (symbol (lib_id "power:-5V") (at 71.12 43.18 0) (unit 1)
-    (in_bom yes) (on_board yes) (fields_autoplaced)
-    (property "Reference" "#PWR?" (id 0) (at 71.12 40.64 0)
-      (effects (font (size 1.27 1.27)) hide)
-    )
-    (property "Value" "-5V" (id 1) (at 71.12 38.1 0))
-    (property "Footprint" "" (id 2) (at 71.12 43.18 0)
-      (effects (font (size 1.27 1.27)) hide)
-    )
-    (property "Datasheet" "" (id 3) (at 71.12 43.18 0)
+  (symbol (lib_id "power:-5V") (at 92.71 52.07 0) (unit 1)
+    (in_bom yes) (on_board yes) (fields_autoplaced)
+    (property "Reference" "#PWR?" (id 0) (at 92.71 49.53 0)
+      (effects (font (size 1.27 1.27)) hide)
+    )
+    (property "Value" "-5V" (id 1) (at 92.71 46.99 0))
+    (property "Footprint" "" (id 2) (at 92.71 52.07 0)
+      (effects (font (size 1.27 1.27)) hide)
+    )
+    (property "Datasheet" "" (id 3) (at 92.71 52.07 0)
       (effects (font (size 1.27 1.27)) hide)
     )
@@
       (reference "#PWR?") (unit 1) (value "+5V") (footprint "")
     )
+    (path "/a9efbe99-7f1b-48c4-a3bf-90bf34e7db79"
+      (reference "#PWR?") (unit 1) (value "GND") (footprint "")
+    )
     (path "/c00ec885-b1f2-44ea-9adc-dbb069945dd6"
       (reference "#PWR?") (unit 1) (value "GND") (footprint "")
@@
       (reference "#PWR?") (unit 1) (value "-5V") (footprint "")
     )
+    (path "/2aa3fdf5-01fd-4ef0-b076-ad9e06ea8d8b"
+      (reference "C1") (unit 1) (value "10pF") (footprint "")
+    )
     (path "/be2a1851-8b8c-4522-94a5-1244e1a2e641"
       (reference "J1") (unit 1) (value "Vin") (footprint "")
     )
+    (path "/1cc9590d-07e5-463e-870e-bee8d9e0235d"
+      (reference "J2") (unit 1) (value "Output") (footprint "")
+    )
     (path "/7420e087-a7b3-4c3c-a4fc-a87f9dad6cbe"
       (reference "R1") (unit 1) (value "9.8k") (footprint "")
@@
       (reference "R4") (unit 1) (value "2k") (footprint "")
     )
+    (path "/386a742f-6f1c-423f-bbed-82e2c21eac3c"
+      (reference "R5") (unit 1) (value "100k") (footprint "")
+    )
     (path "/46da8343-8f47-4fef-90fd-55b846b8bbea"
